File: Plates/wren-nav-top/wren-nav.kicad_pcb (KiCad board)
At the start: 2 copper layers, 201 x 112.8 mm, 46 parts

Commit message: Create .svg for top plates
On realizing that my PCB plates weren't really manufacturable, I decided to use those KiCad files to make a .svg of my plate design that could be laser cut by services like SendCutSend.
Parts:
- removed MX41: MX-NoLED, footprints:MX_Switch_Cutout
- MX1, MX11, MX12, MX13, MX14, MX15, MX16, MX17, MX18, MX19, MX2, MX21, MX22, MX23, MX24, MX25, MX26, MX28, MX3, MX31, MX32, MX33, MX34, MX35, MX36, MX37, MX38, MX39, MX4, MX42, MX43, MX44, MX5, MX6, MX7, MX8, MX9: footprint footprints:MX_Switch_Cutout -> footprints:MX-Alps_Switch_Cutout
- REF**: value MX_Stabilizer_Cutout-2u -> MX-Alps_Switch_Cutout; footprint footprints:MX_Stabilizer_Cutout-2u -> footprints:MX-Alps_Switch_Cutout-1u_2u
